File: essence-pcb-rev_1.kicad_pcb (KiCad board)
At the start: 2 copper layers, 131 parts, among them SW1 Rotary_Encoder_Switch, U1 Elite-C

Commit message: More PCB progress
Parts:
- moved MX-131 197.6 mm to (279.4, 41.3)
- moved MX-12 195.8 mm to (41.3, 60.3)
- moved MX-11 173.4 mm to (41.3, 41.3)
- moved MX-21 166.5 mm to (60.3, 41.3)
- moved MX-22 157.4 mm to (60.3, 60.3)
- moved MX-121 156.4 mm to (250.8, 41.3)
- moved MX-32 154.7 mm to (79.4, 60.3)
- moved MX-91 149.6 mm to (193.7, 41.3)
- moved MX-64 147.3 mm to (-40.5, 69.1)
- moved MX-31 146.2 mm to (79.4, 41.3)
- moved MX-94 144.5 mm to (-15.1, 60.3)
- moved MX-72 133.7 mm to (155.6, 60.3)
- moved MX-51 129.6 mm to (117.5, 41.3)
- moved MX-111 126.8 mm to (231.8, 41.3)
- moved MX-42 114.1 mm to (98.4, 60.3)
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
Commit message: Temporary key grid made
Parts:
- moved MX-133 298.7 mm to (277.0, 79.4)
- moved MX-132 288.1 mm to (281.8, 60.3)
- moved MX-134 248.3 mm to (272.3, 98.4)
- moved MX-94 226.5 mm to (203.2, 120.7)
- moved MX-13 211.5 mm to (41.3, 79.4)
- moved MX-122 191.4 mm to (250.8, 60.3)
- moved MX-64 174.7 mm to (130.2, 106.4)
- moved MX-102 167.0 mm to (212.7, 60.3)
- moved MX-23 160.4 mm to (60.3, 79.4)
- moved MX-104 154.3 mm to (203.2, 101.6)
- moved MX-123 127.4 mm to (250.8, 79.4)
- moved MX-44 125.7 mm to (89.7, 120.7)
- moved MX-84 117.9 mm to (181.8, 111.1)
- moved MX-113 115.6 mm to (231.8, 79.4)
- moved MX-33 115.0 mm to (79.4, 79.4)
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Changed lines of the file:
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@@
     (pad_to_mask_clearance 0)
     (aux_axis_origin 0 0)
-    (visible_elements 7FFFFFFF)
+    (visible_elements 7FFFF7FF)
     (pcbplotparams
       (layerselection 0x010fc_ffffffff)
@@
   )
   (module Keebio-Parts:Elite-C-castellated-29pin-holes (layer F.Cu)
-    (at 38.11275 84.461749)
+    (at 66.675 -12.7)
     (fp_text reference U1 (at 0 1.625) (layer F.SilkS) hide
       (effects (font (size 1.2 1.2) (thickness 0.2032)))
@@
   )
   (module MX_Alps_Hybrid:MX-1.25U-NoLED (layer F.Cu)
-    (at 30.69 155.99875)
+    (at 272.25625 98.425)
     (fp_text reference MX-134 (at 0 3.175) (layer Dwgs.User)
       (effects (font (size 1 1) (thickness 0.15)))
@@
   )
   (module MX_Alps_Hybrid:MX-1.75U-NoLED (layer F.Cu)
-    (at -19.05 39.6875)
+    (at 277.01875 79.375)
     (fp_text reference MX-133 (at 0 3.175) (layer Dwgs.User)
       (effects (font (size 1 1) (thickness 0.15)))
@@
   )
   (module MX_Alps_Hybrid:MX-2.25U-NoLED (layer F.Cu)
-    (at -5.55625 80.9625)
+    (at 281.78125 60.325)
     (fp_text reference MX-132 (at 0 3.175) (layer Dwgs.User)
       (effects (font (size 1 1) (thickness 0.15)))
@@
   )
   (module MX_Alps_Hybrid:MX-1U-NoLED (layer F.Cu)
-    (at 154.26875 162.55875)
+    (at 250.825 79.375)
     (fp_text reference MX-123 (at 0 3.175) (layer Dwgs.User)
       (effects (font (size 1 1) (thickness 0.15)))
@@
   )
   (module MX_Alps_Hybrid:MX-1U-NoLED (layer F.Cu)
-    (at 73.46875 132.31875)
+    (at 250.825 60.325)
     (fp_text reference MX-122 (at 0 3.175) (layer Dwgs.User)
       (effects (font (size 1 1) (thickness 0.15)))
@@
   )
   (module MX_Alps_Hybrid:MX-1U-NoLED (layer F.Cu)
-    (at 148.43125 -0.79375)
+    (at 231.775 79.375)
     (fp_text reference MX-113 (at 0 3.175) (layer Dwgs.User)
       (effects (font (size 1 1) (thickness 0.15)))
@@
   )
   (module MX_Alps_Hybrid:MX-1U-NoLED (layer F.Cu)
-    (at 231.775 -2.38125)
+    (at 231.775 60.325)
     (fp_text reference MX-112 (at 0 3.175) (layer Dwgs.User)
       (effects (font (size 1 1) (thickness 0.15)))
@@
   )
   (module MX_Alps_Hybrid:MX-1.25U-NoLED (layer F.Cu)
-    (at 50.89 126.27875)
+    (at 203.2 101.6)
     (fp_text reference MX-104 (at 0 3.175) (layer Dwgs.User)
       (effects (font (size 1 1) (thickness 0.15)))
@@
   )
   (module MX_Alps_Hybrid:MX-1U-NoLED (layer F.Cu)
-    (at 131.56875 81.75875)
+    (at 212.725 79.375)
     (fp_text reference MX-103 (at 0 3.175) (layer Dwgs.User)
       (effects (font (size 1 1) (thickness 0.15)))
@@
   )
   (module MX_Alps_Hybrid:MX-1U-NoLED (layer F.Cu)
-    (at 73.46875 152.51875)
+    (at 212.725 60.325)
     (fp_text reference MX-102 (at 0 3.175) (layer Dwgs.User)
       (effects (font (size 1 1) (thickness 0.15)))
@@
   )
   (module MX_Alps_Hybrid:MX-1.25U-NoLED (layer F.Cu)
-    (at -15.08125 60.325)
+    (at 203.2 120.65)
     (fp_text reference MX-94 (at 0 3.175) (layer Dwgs.User)
       (effects (font (size 1 1) (thickness 0.15)))
@@
   )
   (module MX_Alps_Hybrid:MX-1U-NoLED (layer F.Cu)
-    (at 131.56875 101.95875)
+    (at 193.675 79.375)
     (fp_text reference MX-93 (at 0 3.175) (layer Dwgs.User)
       (effects (font (size 1 1) (thickness 0.15)))
@@
   )
   (module MX_Alps_Hybrid:MX-1.5U-Vertical (layer F.Cu)
-    (at 66.20875 87.80125)
+    (at 181.76875 111.125)
     (fp_text reference MX-84 (at 0 3.175) (layer Dwgs.User)
       (effects (font (size 1 1) (thickness 0.15)))
@@
   )
   (module MX_Alps_Hybrid:MX-1U-NoLED (layer F.Cu)
-    (at 201.6125 -0.79375)
+    (at 174.625 79.375)
     (fp_text reference MX-83 (at 0 3.175) (layer Dwgs.User)
       (effects (font (size 1 1) (thickness 0.15)))
@@
   )
   (module MX_Alps_Hybrid:MX-1.5U-Vertical (layer F.Cu)
-    (at 86.40875 87.16125)
+    (at 162.71875 106.3625)
     (fp_text reference MX-74 (at 0 3.175) (layer Dwgs.User)
       (effects (font (size 1 1) (thickness 0.15)))
@@
   )
   (module MX_Alps_Hybrid:MX-1.5U-Vertical (layer F.Cu)
-    (at -40.48125 69.05625)
+    (at 130.175 106.3625)
     (fp_text reference MX-64 (at 0 3.175) (layer Dwgs.User)
       (effects (font (size 1 1) (thickness 0.15)))
@@
   )
   (module MX_Alps_Hybrid:MX-1.5U-Vertical (layer F.Cu)
-    (at 28.30875 131.04125)
+    (at 111.125 111.125)
     (fp_text reference MX-54 (at 0 3.175) (layer Dwgs.User)
       (effects (font (size 1 1) (thickness 0.15)))
@@
   )
   (module MX_Alps_Hybrid:MX-1U-NoLED (layer F.Cu)
-    (at 212.36875 81.75875)
+    (at 117.475 79.375)
     (fp_text reference MX-53 (at 0 3.175) (layer Dwgs.User)
       (effects (font (size 1 1) (thickness 0.15)))
@@
   )
   (module MX_Alps_Hybrid:MX-1.25U-NoLED (layer F.Cu)
-    (at 122.2375 -0.79375)
+    (at 89.69375 120.65)
     (fp_text reference MX-44 (at 0 3.175) (layer Dwgs.User)
       (effects (font (size 1 1) (thickness 0.15)))
@@
   )
   (module MX_Alps_Hybrid:MX-1U-NoLED (layer F.Cu)
-    (at 154.26875 122.15875)
+    (at 98.425 79.375)
     (fp_text reference MX-43 (at 0 3.175) (layer Dwgs.User)
       (effects (font (size 1 1) (thickness 0.15)))
@@
   )
   (module MX_Alps_Hybrid:MX-1.25U-NoLED (layer F.Cu)
-    (at 88.79 112.11875)
+    (at 89.69375 101.6)
     (fp_text reference MX-34 (at 0 3.175) (layer Dwgs.User)
       (effects (font (size 1 1) (thickness 0.15)))
@@
   )
   (module MX_Alps_Hybrid:MX-1U-NoLED (layer F.Cu)
-    (at 192.16875 101.95875)
+    (at 79.375 79.375)
     (fp_text reference MX-33 (at 0 3.175) (layer Dwgs.User)
       (effects (font (size 1 1) (thickness 0.15)))
@@
   )
   (module MX_Alps_Hybrid:MX-1U-NoLED (layer F.Cu)
-    (at 214.86875 122.15875)
+    (at 60.325 79.375)
     (fp_text reference MX-23 (at 0 3.175) (layer Dwgs.User)
       (effects (font (size 1 1) (thickness 0.15)))
@@
   )
   (module MX_Alps_Hybrid:MX-1U-NoLED (layer F.Cu)
-    (at 252.76875 81.75875)
+    (at 41.275 79.375)
     (fp_text reference MX-13 (at 0 3.175) (layer Dwgs.User)
       (effects (font (size 1 1) (thickness 0.15)))
@@
   )
   (module MX_Alps_Hybrid:MX-1.25U-NoLED (layer F.Cu)
-    (at 108.99 91.91875)
+    (at 19.84375 98.425)
     (fp_text reference MX-4 (at 0 3.175) (layer Dwgs.User)
       (effects (font (size 1 1) (thickness 0.15)))
@@
   )
   (module MX_Alps_Hybrid:MX-2.25U-NoLED (layer F.Cu)
-    (at 0.79375 -3.96875)
+    (at 10.31875 79.375)
     (fp_text reference MX-3 (at 0 3.175) (layer Dwgs.User)
       (effects (font (size 1 1) (thickness 0.15)))
@@
   )
   (module Diode_THT:D_DO-35_SOD27_P7.62mm_Horizontal (layer F.Cu)
-    (at 264.44375 73.43375)
+    (at 293.8125 13.10875)
     (descr "Diode, DO-35_SOD27 series, Axial, Horizontal, pin pitch=7.62mm, , length*diameter=4*2mm^2, , http://www.diodes.com/_files/packages/DO-35.pdf")
     (tags "Diode DO-35_SOD27 series Axial Horizontal pin pitch 7.62mm  length 4mm diameter 2mm")
@@
   )
   (module Diode_THT:D_DO-35_SOD27_P7.62mm_Horizontal (layer F.Cu)
-    (at 275.21375 73.43375)
+    (at 304.5825 13.10875)
     (descr "Diode, DO-35_SOD27 series, Axial, Horizontal, pin pitch=7.62mm, , length*diameter=4*2mm^2, , http://www.diodes.com/_files/packages/DO-35.pdf")
     (tags "Diode DO-35_SOD27 series Axial Horizontal pin pitch 7.62mm  length 4mm diameter 2mm")
@@
   )
   (module Diode_THT:D_DO-35_SOD27_P7.62mm_Horizontal (layer F.Cu)
-    (at 264.44375 76.98375)
+    (at 293.8125 16.65875)
     (descr "Diode, DO-35_SOD27 series, Axial, Horizontal, pin pitch=7.62mm, , length*diameter=4*2mm^2, , http://www.diodes.com/_files/packages/DO-35.pdf")
     (tags "Diode DO-35_SOD27 series Axial Horizontal pin pitch 7.62mm  length 4mm diameter 2mm")
@@
   )
   (module Diode_THT:D_DO-35_SOD27_P7.62mm_Horizontal (layer F.Cu)
-    (at 264.44375 80.53375)
+    (at 293.8125 20.20875)
     (descr "Diode, DO-35_SOD27 series, Axial, Horizontal, pin pitch=7.62mm, , length*diameter=4*2mm^2, , http://www.diodes.com/_files/packages/DO-35.pdf")
     (tags "Diode DO-35_SOD27 series Axial Horizontal pin pitch 7.62mm  length 4mm diameter 2mm")
@@
   )
   (module Diode_THT:D_DO-35_SOD27_P7.62mm_Horizontal (layer F.Cu)
-    (at 264.44375 84.08375)
+    (at 293.8125 23.75875)
     (descr "Diode, DO-35_SOD27 series, Axial, Horizontal, pin pitch=7.62mm, , length*diameter=4*2mm^2, , http://www.diodes.com/_files/packages/DO-35.pdf")
     (tags "Diode DO-35_SOD27 series Axial Horizontal pin pitch 7.62mm  length 4mm diameter 2mm")

Commit message: Ergolinear format for left side
Parts:
- moved U1 85.2 mm to (150.0, -30.2), turned to 270 degrees
- moved D10 29.1 mm to (317.3, 39.3)
- moved MX-131 29.1 mm to (292.1, 67.5)
- moved D31 29.1 mm to (239.2, 150.7)
- moved D52 29.1 mm to (239.2, 140.0)
- moved MX-104 29.1 mm to (215.9, 127.8)
- moved MX-100 29.1 mm to (225.4, 48.4)
- moved MX-101 29.1 mm to (225.4, 67.5)
- moved MX-70 29.1 mm to (168.3, 48.4)
- moved MX-71 29.1 mm to (168.3, 67.5)
- moved D1 29.1 mm to (250.0, 140.0)
- moved MX-134 29.1 mm to (285.0, 124.6)
- moved MX-74 29.1 mm to (175.4, 132.6)
- moved D3 29.1 mm to (306.5, 46.4)
- moved D32 29.1 mm to (239.2, 147.1)
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
Commit message: Non-tented layout finished
Parts:
- moved D2 284.5 mm to (23.0, 26.2)
- moved D3 284.0 mm to (23.0, 29.4)
- moved D4 283.7 mm to (23.0, 32.5)
- moved D1 255.4 mm to (23.0, 23.0)
- moved D0 191.2 mm to (23.0, 19.8)
- moved MX-100 22.0 mm to (242.1, 34.1)
- moved MX-101 22.0 mm to (242.1, 53.2)
- moved MX-102 22.0 mm to (242.1, 72.2)
- moved MX-103 22.0 mm to (242.1, 91.3)
- moved MX-110 19.2 mm to (261.1, 38.9)
- moved MX-111 19.2 mm to (261.1, 57.9)
- moved MX-112 19.2 mm to (261.1, 77.0)
- moved MX-113 19.2 mm to (261.1, 96.0)
- moved MX-90 19.2 mm to (223.0, 38.9)
- moved MX-91 19.2 mm to (223.0, 57.9)
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
Commit message: Diode proximity established
Parts:
- moved D130 306.5 mm to (295.3, 36.5)
- moved D10 295.9 mm to (38.1, 31.8)
- moved D131 274.1 mm to (305.6, 57.9)
- moved D132 270.9 mm to (292.9, 84.9)
- moved D134 246.9 mm to (298.4, 115.1)
- moved D120 245.2 mm to (276.2, 31.8)
- moved D133 242.8 mm to (290.5, 102.4)
- moved D41 228.1 mm to (95.2, 48.4)
- moved D121 227.5 mm to (277.0, 53.2)
- moved D110 227.1 mm to (257.2, 27.0)
- moved D101 226.3 mm to (238.9, 43.7)
- moved D100 226.1 mm to (238.1, 22.2)
- moved D122 222.3 mm to (277.0, 72.2)
- moved D90 218.5 mm to (219.1, 27.0)
- moved D123 218.0 mm to (277.0, 91.3)
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
Commit message: PCB tent integrated
For some reason, multi-footprint rotate is located in the move window? If you are reading this go make a milkshake
Parts:
- moved D40 85.1 mm to (172.4, 62.8), turned to 255 degrees
- moved D60 85.1 mm to (208.0, 77.3), turned to 255 degrees
- moved D30 85.0 mm to (155.3, 53.3), turned to 255 degrees
- moved D50 84.9 mm to (189.6, 72.4), turned to 255 degrees
- moved D20 82.5 mm to (136.9, 48.4), turned to 255 degrees
- moved D10 80.8 mm to (117.2, 48.0), turned to 255 degrees
- moved D41 79.4 mm to (167.5, 81.2), turned to 255 degrees
- moved D0 79.4 mm to (97.6, 47.7), turned to 255 degrees
- moved D31 79.3 mm to (150.3, 71.7), turned to 255 degrees
- moved D51 79.1 mm to (184.7, 90.8), turned to 255 degrees
- moved D61 78.6 mm to (203.1, 95.7), turned to 255 degrees
- moved D21 76.2 mm to (131.9, 66.8), turned to 255 degrees
- moved MX-74 74.9 mm to (247.2, 158.1), turned to 15 degrees
- moved D11 74.6 mm to (112.3, 66.4), turned to 255 degrees
- moved D52 74.5 mm to (179.8, 109.2), turned to 255 degrees
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
Commit message: Elite C positioned in center
This may be changed depending on cable position preferences, will sleep on it.
Parts:
- moved U1 102.1 mm to (214.3, 49.2)
Changed lines of the file:
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@@
   )
   (module Keebio-Parts:Elite-C-castellated-29pin-holes (layer F.Cu)
-    (at 150.01875 -30.1625 270)
+    (at 214.3125 49.2125 270)
     (fp_text reference U1 (at 0 1.625 90) (layer F.SilkS) hide
       (effects (font (size 1.2 1.2) (thickness 0.2032)))

Commit message: Board Outline made
Other:
- board outline added: 352.4 x 144.5 mm
