File: essence-pcb-rev_1.kicad_pcb (KiCad board)
At the start: 2 copper layers, 352.4 x 144.5 mm, 131 parts, among them SW1 Rotary_Encoder_Switch, U1 Elite-C

Commit message: Initial routing pattern
Routing:
- net Row4: track 0.00 -> 318.9 mm
- net Row3: track 0.00 -> 307.8 mm
- net Row2: track 0.00 -> 291.3 mm
- net Row1: track 0.00 -> 276.2 mm
- net Row0: track 0.00 -> 262.3 mm
- net Col7: track 0.00 -> 120.4 mm
- net Col9: track 0.00 -> 107.9 mm
- net Col4: track 0.00 -> 103.0 mm
- net Col3: track 0.00 -> 102.7 mm
- net Col10: track 0.00 -> 97.0 mm
- net Col8: track 0.00 -> 88.6 mm
- net Col0: track 0.00 -> 86.2 mm
- net Col5: track 0.00 -> 86.1 mm
- net Col13: track 0.00 -> 80.0 mm
- net Col6: track 0.00 -> 79.3 mm
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
Commit message: Updated pin placement on Elite C to matrix
Connections:
- U1 pad 10: Col3 -> Col5
- U1 pad 11: Col4 -> Row0
- U1 pad 12: Col5 -> Row1
- U1 pad 13: Col13 -> Col6
- U1 pad 14: Col12 -> Col7
- U1 pad 15: Col11 -> Col8
- U1 pad 16: Col10 -> Col9
- U1 pad 17: Col9 -> Col10
- U1 pad 18: Col8 -> Col11
- U1 pad 19: Col7 -> Col12
- U1 pad 20: Col6 -> Col13
- U1 pad 25: Row4 -> Row2
- U1 pad 27: Row2 -> Row4
- U1 pad 28: Row1 -> Enc1
- U1 pad 29: Row0 -> Enc0
- U1 pad 5: Enc0 -> Col0
- U1 pad 6: Enc1 -> Col1
- U1 pad 7: Col0 -> Col2
- U1 pad 8: Col1 -> Col3
- U1 pad 9: Col2 -> Col4

Commit message: Track Rough Draft (all connected, edit needed)
Connections:
- U1 pad 11: Row0 -> Col6
- U1 pad 12: Row1 -> Row0
- U1 pad 13: Col6 -> Enc0
- U1 pad 25: Row2 -> Row1
- U1 pad 26: Row3 -> Row2
- U1 pad 27: Row4 -> Row3
- U1 pad 28: Enc1 -> Row4
- U1 pad 29: Enc0 -> Enc1
Routing:
- net Col0: track 86.2 -> 213.2 mm
- net Col13: track 80.0 -> 201.1 mm
- net Col1: track 64.0 -> 171.3 mm
- net Row4: track 318.9 -> 420.5 mm
- net Col12: track 58.6 -> 159.0 mm
- net Row3: track 307.8 -> 400.5 mm, vias 0 -> 1
- net Col2: track 62.2 -> 150.4 mm
- net Col11: track 57.2 -> 138.8 mm
- net Col3: track 102.7 -> 170.0 mm
- net Enc0: track 0.00 -> 64.1 mm
- net Enc1: track 0.00 -> 62.6 mm
- net Col10: track 97.0 -> 156.9 mm
- net Row2: track 291.3 -> 347.9 mm
- net Col4: track 103.0 -> 152.6 mm
- net Col9: track 107.9 -> 151.0 mm
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
Commit message: Final Routing
Routing:
- net Col0: track 213.2 -> 223.9 mm
- net Col7: track 146.1 -> 138.2 mm
- net Col13: track 201.1 -> 206.2 mm
- net Col1: track 171.3 -> 175.2 mm
- net Row4: track 420.5 -> 417.8 mm
- net Col9: track 151.0 -> 153.4 mm
- net Col10: track 156.9 -> 159.0 mm
- net Col12: track 159.0 -> 160.8 mm
- net Col2: track 150.4 -> 152.0 mm
- net Col4: track 152.6 -> 153.4 mm
- net Col8: track 117.4 -> 118.0 mm

Commit message: Reset Switch added, and Ground fields defined
I think I outlined the ground fields correctly, but I will get input to be sure before I manufacture it
Parts:
- added SW-Rst1: SW_Push, Keebio-Parts:SW_Tactile_SPST_Angled_MJTP1117, F.Cu at (244.5, 44.5)
Connections:
- U1 pad 23: Net-(U1-Pad23) -> GND
- U1 pad 3: Net-(U1-Pad3) -> GND
- U1 pad 4: Net-(U1-Pad4) -> GND
Routing:
- net GND: track 0.00 -> 152.5 mm, vias 0 -> 1
- net Net-(SW-Rst1-Pad1): track 0.00 -> 24.8 mm
- net Col13: track 206.2 -> 213.8 mm
- net Col12: track 160.8 -> 167.4 mm
- net Col11: track 138.8 -> 143.5 mm
- net Col10: track 159.0 -> 162.2 mm
- added copper zone on B.Cu, net GND
- added copper zone on F.Cu, net GND

Commit message: PCB graphics
Parts:
- added G***: LOGO, random-keyboard-parts:Logo_Nite, B.Cu at (215.9, 165.1)
- added G***: LOGO, random-keyboard-parts:Logo_ObamaPrism3, F.Cu at (218.3, 115.9)
- added G***: LOGO, random-keyboard-parts:Logo_GigaChad, B.Cu at (215.1, 100.0)
Other:
- board text added: "Created for SHS Senior Project, 2022"
- board text added: "Designed by Hyper-works, circa March 2022"
- board text added: "Essence Ergo Keyboard Model 0.0"
